Commit message: support better scout v2 simulation

File: scout/scout_description/urdf/scout_v2.xacro (robot description, xacro)
@@ -84,3 +84,7 @@
     <!-- Gazebo definitions  -->
     <xacro:include filename="$(find scout_description)/urdf/scout_v2.gazebo" />
+  <xacro:include filename="$(find robosense_description)/urdf/RS-16.urdf.xacro"/>
+  <xacro:RS-16 parent="base_link" name="robosense" topic="/rslidar_points" hz="20" samples="900" gpu="false">
+    <origin xyz="0 0 0.4" rpy="0 0 0" />
+  </xacro:RS-16>
 </robot>

Commit message: adjust lidar pose

File: scout/scout_description/urdf/scout_v2.xacro (robot description, xacro)
@@ -86,5 +86,5 @@
   <xacro:include filename="$(find robosense_description)/urdf/RS-16.urdf.xacro"/>
   <xacro:RS-16 parent="base_link" name="robosense" topic="/rslidar_points" hz="20" samples="900" gpu="false">
-    <origin xyz="0 0 0.4" rpy="0 0 0" />
+    <origin xyz="0.35 0 0.4" rpy="0 0 0" />
   </xacro:RS-16>
 </robot>

Commit message: add depth camera

File: scout/scout_description/urdf/scout_v2.xacro (robot description, xacro)
@@ -84,7 +84,11 @@
     <!-- Gazebo definitions  -->
     <xacro:include filename="$(find scout_description)/urdf/scout_v2.gazebo" />
-  <xacro:include filename="$(find robosense_description)/urdf/RS-16.urdf.xacro"/>
-  <xacro:RS-16 parent="base_link" name="robosense" topic="/rslidar_points" hz="20" samples="900" gpu="false">
-    <origin xyz="0.35 0 0.4" rpy="0 0 0" />
-  </xacro:RS-16>
+    <xacro:include filename="$(find robosense_description)/urdf/RS-16.urdf.xacro"/>
+    <xacro:RS-16 parent="base_link" name="robosense" topic="/rslidar_points" hz="20" samples="900" gpu="false">
+        <origin xyz="0.35 0 0.4" rpy="0 0 0" />
+    </xacro:RS-16>
+    <xacro:include filename="$(find realsense_ros_gazebo)/xacro/depthcam.xacro"/>
+    <xacro:realsense_R200 sensor_name="camera" parent_link="base_link" rate="30.0">
+        <origin rpy="0 0 1.5708" xyz="0 0 0.5"/>
+    </xacro:realsense_R200>
 </robot>

Commit message: add camera to scout v2 and change back world file

File: scout/scout_description/urdf/scout_v2.xacro (robot description, xacro)
@@ -86,9 +86,14 @@
     <xacro:include filename="$(find robosense_description)/urdf/RS-16.urdf.xacro"/>
     <xacro:RS-16 parent="base_link" name="robosense" topic="/rslidar_points" hz="20" samples="900" gpu="false">
-        <origin xyz="0.35 0 0.4" rpy="0 0 0" />
+        <!-- <origin xyz="0.35 0 0.4" rpy="0 0 0" /> -->
+        <origin xyz="0.35 0 0.2" rpy="0 0 0" />
     </xacro:RS-16>
+    <!-- <xacro:include filename="$(find realsense_ros_gazebo)/xacro/depthcam.xacro"/>
+    <xacro:realsense_R200 sensor_name="camera" parent_link="base_link" rate="30.0">
+        <origin rpy="0 0 1.5708" xyz="0 0 0.5"/>
+    </xacro:realsense_R200> -->
     <xacro:include filename="$(find realsense_ros_gazebo)/xacro/depthcam.xacro"/>
     <xacro:realsense_R200 sensor_name="camera" parent_link="base_link" rate="30.0">
-        <origin rpy="0 0 1.5708" xyz="0 0 0.5"/>
+        <origin rpy="0 0 0" xyz="0 0 0.5"/>
     </xacro:realsense_R200>
 </robot>
